Commit message: pakage

File: src/nhk2026_sim/urdf/robot.xacro (robot description, xacro)
@@ -13,5 +13,5 @@
     <origin xyz="0 0 0" rpy="0 0 0"/>
     <geometry>
-      <mesh filename="file://$(find nhk2026_sim)/meshes/base_link.stl" scale="0.001 0.001 0.001"/>
+      <mesh filename="package://nhk2026_sim/meshes/base_link.stl" scale="0.001 0.001 0.001"/>
     </geometry>
     <material name="steel_satin"/>
@@ -20,5 +20,5 @@
     <origin xyz="0 0 0" rpy="0 0 0"/>
     <geometry>
-      <mesh filename="file://$(find nhk2026_sim)/meshes/base_link.stl" scale="0.001 0.001 0.001"/>
+      <mesh filename="package://nhk2026_sim/meshes/base_link.stl" scale="0.001 0.001 0.001"/>
     </geometry>
   </collision>
@@ -33,5 +33,5 @@
     <origin xyz="-0.007243 -0.081923 0.003" rpy="0 0 0"/>
     <geometry>
-      <mesh filename="file://$(find nhk2026_sim)/meshes/alm_1_v4_1.stl" scale="0.001 0.001 0.001"/>
+      <mesh filename="package://nhk2026_sim/meshes/alm_1_v4_1.stl" scale="0.001 0.001 0.001"/>
     </geometry>
     <material name="aluminum_satin"/>
@@ -40,5 +40,5 @@
     <origin xyz="-0.007243 -0.081923 0.003" rpy="0 0 0"/>
     <geometry>
-      <mesh filename="file://$(find nhk2026_sim)/meshes/alm_1_v4_1.stl" scale="0.001 0.001 0.001"/>
+      <mesh filename="package://nhk2026_sim/meshes/alm_1_v4_1.stl" scale="0.001 0.001 0.001"/>
     </geometry>
   </collision>
@@ -53,5 +53,5 @@
     <origin xyz="-0.020233 -0.089423 0.013" rpy="0 0 0"/>
     <geometry>
-      <mesh filename="file://$(find nhk2026_sim)/meshes/chassis_unit_v18_1.stl" scale="0.001 0.001 0.001"/>
+      <mesh filename="package://nhk2026_sim/meshes/chassis_unit_v18_1.stl" scale="0.001 0.001 0.001"/>
     </geometry>
     <material name="steel_satin"/>
@@ -60,5 +60,5 @@
     <origin xyz="-0.020233 -0.089423 0.013" rpy="0 0 0"/>
     <geometry>
-      <mesh filename="file://$(find nhk2026_sim)/meshes/chassis_unit_v18_1.stl" scale="0.001 0.001 0.001"/>
+      <mesh filename="package://nhk2026_sim/meshes/chassis_unit_v18_1.stl" scale="0.001 0.001 0.001"/>
     </geometry>
   </collision>
@@ -73,5 +73,5 @@
     <origin xyz="-0.072195 -0.059423 0.013" rpy="0 0 0"/>
     <geometry>
-      <mesh filename="file://$(find nhk2026_sim)/meshes/alm_with_lidar_v6_1.stl" scale="0.001 0.001 0.001"/>
+      <mesh filename="package://nhk2026_sim/meshes/alm_with_lidar_v6_1.stl" scale="0.001 0.001 0.001"/>
     </geometry>
     <material name="aluminum_satin"/>
@@ -80,5 +80,5 @@
     <origin xyz="-0.072195 -0.059423 0.013" rpy="0 0 0"/>
     <geometry>
-      <mesh filename="file://$(find nhk2026_sim)/meshes/alm_with_lidar_v6_1.stl" scale="0.001 0.001 0.001"/>
+      <mesh filename="package://nhk2026_sim/meshes/alm_with_lidar_v6_1.stl" scale="0.001 0.001 0.001"/>
     </geometry>
   </collision>
@@ -93,5 +93,5 @@
     <origin xyz="-0.072195 0.060577 0.013" rpy="0 0 0"/>
     <geometry>
-      <mesh filename="file://$(find nhk2026_sim)/meshes/chassis_unit_v18_2.stl" scale="0.001 0.001 0.001"/>
+      <mesh filename="package://nhk2026_sim/meshes/chassis_unit_v18_2.stl" scale="0.001 0.001 0.001"/>
     </geometry>
     <material name="steel_satin"/>
@@ -100,5 +100,5 @@
     <origin xyz="-0.072195 0.060577 0.013" rpy="0 0 0"/>
     <geometry>
-      <mesh filename="file://$(find nhk2026_sim)/meshes/chassis_unit_v18_2.stl" scale="0.001 0.001 0.001"/>
+      <mesh filename="package://nhk2026_sim/meshes/chassis_unit_v18_2.stl" scale="0.001 0.001 0.001"/>
     </geometry>
   </collision>
@@ -113,5 +113,5 @@
     <origin xyz="-0.020233 0.090577 0.013" rpy="0 0 0"/>
     <geometry>
-      <mesh filename="file://$(find nhk2026_sim)/meshes/alm_1_v4_2.stl" scale="0.001 0.001 0.001"/>
+      <mesh filename="package://nhk2026_sim/meshes/alm_1_v4_2.stl" scale="0.001 0.001 0.001"/>
     </geometry>
     <material name="aluminum_satin"/>
@@ -120,5 +120,5 @@
     <origin xyz="-0.020233 0.090577 0.013" rpy="0 0 0"/>
     <geometry>
-      <mesh filename="file://$(find nhk2026_sim)/meshes/alm_1_v4_2.stl" scale="0.001 0.001 0.001"/>
+      <mesh filename="package://nhk2026_sim/meshes/alm_1_v4_2.stl" scale="0.001 0.001 0.001"/>
     </geometry>
   </collision>
@@ -133,5 +133,5 @@
     <origin xyz="0.08369 -0.029423 0.013" rpy="0 0 0"/>
     <geometry>
-      <mesh filename="file://$(find nhk2026_sim)/meshes/chassis_unit_v18_3.stl" scale="0.001 0.001 0.001"/>
+      <mesh filename="package://nhk2026_sim/meshes/chassis_unit_v18_3.stl" scale="0.001 0.001 0.001"/>
     </geometry>
     <material name="steel_satin"/>
@@ -140,5 +140,5 @@
     <origin xyz="0.08369 -0.029423 0.013" rpy="0 0 0"/>
     <geometry>
-      <mesh filename="file://$(find nhk2026_sim)/meshes/chassis_unit_v18_3.stl" scale="0.001 0.001 0.001"/>
+      <mesh filename="package://nhk2026_sim/meshes/chassis_unit_v18_3.stl" scale="0.001 0.001 0.001"/>
     </geometry>
   </collision>
@@ -153,5 +153,5 @@
     <origin xyz="-0.072195 0.023977 0.013" rpy="0 0 0"/>
     <geometry>
-      <mesh filename="file://$(find nhk2026_sim)/meshes/LD19_with_mounter_v17_1.stl" scale="0.001 0.001 0.001"/>
+      <mesh filename="package://nhk2026_sim/meshes/LD19_with_mounter_v17_1.stl" scale="0.001 0.001 0.001"/>
     </geometry>
     <material name="steel_satin"/>
@@ -160,5 +160,5 @@
     <origin xyz="-0.072195 0.023977 0.013" rpy="0 0 0"/>
     <geometry>
-      <mesh filename="file://$(find nhk2026_sim)/meshes/LD19_with_mounter_v17_1.stl" scale="0.001 0.001 0.001"/>
+      <mesh filename="package://nhk2026_sim/meshes/LD19_with_mounter_v17_1.stl" scale="0.001 0.001 0.001"/>
     </geometry>
   </collision>
@@ -173,5 +173,5 @@
     <origin xyz="0.044719 0.053077 0.013" rpy="0 0 0"/>
     <geometry>
-      <mesh filename="file://$(find nhk2026_sim)/meshes/fun_adapter_v2_1.stl" scale="0.001 0.001 0.001"/>
+      <mesh filename="package://nhk2026_sim/meshes/fun_adapter_v2_1.stl" scale="0.001 0.001 0.001"/>
     </geometry>
     <material name="steel_satin"/>
@@ -180,5 +180,5 @@
     <origin xyz="0.044719 0.053077 0.013" rpy="0 0 0"/>
     <geometry>
-      <mesh filename="file://$(find nhk2026_sim)/meshes/fun_adapter_v2_1.stl" scale="0.001 0.001 0.001"/>
+      <mesh filename="package://nhk2026_sim/meshes/fun_adapter_v2_1.stl" scale="0.001 0.001 0.001"/>
     </geometry>
   </collision>
@@ -193,5 +193,5 @@
     <origin xyz="0.065593 0.061233 0.016" rpy="0 0 0"/>
     <geometry>
-      <mesh filename="file://$(find nhk2026_sim)/meshes/fun_v13_1.stl" scale="0.001 0.001 0.001"/>
+      <mesh filename="package://nhk2026_sim/meshes/fun_v13_1.stl" scale="0.001 0.001 0.001"/>
     </geometry>
     <material name="steel_satin"/>
@@ -200,5 +200,5 @@
     <origin xyz="0.065593 0.061233 0.016" rpy="0 0 0"/>
     <geometry>
-      <mesh filename="file://$(find nhk2026_sim)/meshes/fun_v13_1.stl" scale="0.001 0.001 0.001"/>
+      <mesh filename="package://nhk2026_sim/meshes/fun_v13_1.stl" scale="0.001 0.001 0.001"/>
     </geometry>
   </collision>

Commit message: sim

File: src/nhk2026_sim/urdf/robot.xacro (robot description, xacro)
@@ -13,5 +13,5 @@
     <origin xyz="0 0 0" rpy="0 0 0"/>
     <geometry>
-      <mesh filename="package://nhk2026_sim/meshes/base_link.stl" scale="0.001 0.001 0.001"/>
+      <mesh filename="file://$(find nhk2026_sim)/meshes/base_link.stl" scale="0.001 0.001 0.001"/>
     </geometry>
     <material name="steel_satin"/>
@@ -20,5 +20,5 @@
     <origin xyz="0 0 0" rpy="0 0 0"/>
     <geometry>
-      <mesh filename="package://nhk2026_sim/meshes/base_link.stl" scale="0.001 0.001 0.001"/>
+      <mesh filename="file://$(find nhk2026_sim)/meshes/base_link.stl" scale="0.001 0.001 0.001"/>
     </geometry>
   </collision>
@@ -33,5 +33,5 @@
     <origin xyz="-0.007243 -0.081923 0.003" rpy="0 0 0"/>
     <geometry>
-      <mesh filename="package://nhk2026_sim/meshes/alm_1_v4_1.stl" scale="0.001 0.001 0.001"/>
+      <mesh filename="file://$(find nhk2026_sim)/meshes/alm_1_v4_1.stl" scale="0.001 0.001 0.001"/>
     </geometry>
     <material name="aluminum_satin"/>
@@ -40,5 +40,5 @@
     <origin xyz="-0.007243 -0.081923 0.003" rpy="0 0 0"/>
     <geometry>
-      <mesh filename="package://nhk2026_sim/meshes/alm_1_v4_1.stl" scale="0.001 0.001 0.001"/>
+      <mesh filename="file://$(find nhk2026_sim)/meshes/alm_1_v4_1.stl" scale="0.001 0.001 0.001"/>
     </geometry>
   </collision>
@@ -53,5 +53,5 @@
     <origin xyz="-0.020233 -0.089423 0.013" rpy="0 0 0"/>
     <geometry>
-      <mesh filename="package://nhk2026_sim/meshes/chassis_unit_v18_1.stl" scale="0.001 0.001 0.001"/>
+      <mesh filename="file://$(find nhk2026_sim)/meshes/chassis_unit_v18_1.stl" scale="0.001 0.001 0.001"/>
     </geometry>
     <material name="steel_satin"/>
@@ -60,5 +60,5 @@
     <origin xyz="-0.020233 -0.089423 0.013" rpy="0 0 0"/>
     <geometry>
-      <mesh filename="package://nhk2026_sim/meshes/chassis_unit_v18_1.stl" scale="0.001 0.001 0.001"/>
+      <mesh filename="file://$(find nhk2026_sim)/meshes/chassis_unit_v18_1.stl" scale="0.001 0.001 0.001"/>
     </geometry>
   </collision>
@@ -73,5 +73,5 @@
     <origin xyz="-0.072195 -0.059423 0.013" rpy="0 0 0"/>
     <geometry>
-      <mesh filename="package://nhk2026_sim/meshes/alm_with_lidar_v6_1.stl" scale="0.001 0.001 0.001"/>
+      <mesh filename="file://$(find nhk2026_sim)/meshes/alm_with_lidar_v6_1.stl" scale="0.001 0.001 0.001"/>
     </geometry>
     <material name="aluminum_satin"/>
@@ -80,5 +80,5 @@
     <origin xyz="-0.072195 -0.059423 0.013" rpy="0 0 0"/>
     <geometry>
-      <mesh filename="package://nhk2026_sim/meshes/alm_with_lidar_v6_1.stl" scale="0.001 0.001 0.001"/>
+      <mesh filename="file://$(find nhk2026_sim)/meshes/alm_with_lidar_v6_1.stl" scale="0.001 0.001 0.001"/>
     </geometry>
   </collision>
@@ -93,5 +93,5 @@
     <origin xyz="-0.072195 0.060577 0.013" rpy="0 0 0"/>
     <geometry>
-      <mesh filename="package://nhk2026_sim/meshes/chassis_unit_v18_2.stl" scale="0.001 0.001 0.001"/>
+      <mesh filename="file://$(find nhk2026_sim)/meshes/chassis_unit_v18_2.stl" scale="0.001 0.001 0.001"/>
     </geometry>
     <material name="steel_satin"/>
@@ -100,5 +100,5 @@
     <origin xyz="-0.072195 0.060577 0.013" rpy="0 0 0"/>
     <geometry>
-      <mesh filename="package://nhk2026_sim/meshes/chassis_unit_v18_2.stl" scale="0.001 0.001 0.001"/>
+      <mesh filename="file://$(find nhk2026_sim)/meshes/chassis_unit_v18_2.stl" scale="0.001 0.001 0.001"/>
     </geometry>
   </collision>
@@ -113,5 +113,5 @@
     <origin xyz="-0.020233 0.090577 0.013" rpy="0 0 0"/>
     <geometry>
-      <mesh filename="package://nhk2026_sim/meshes/alm_1_v4_2.stl" scale="0.001 0.001 0.001"/>
+      <mesh filename="file://$(find nhk2026_sim)/meshes/alm_1_v4_2.stl" scale="0.001 0.001 0.001"/>
     </geometry>
     <material name="aluminum_satin"/>
@@ -120,5 +120,5 @@
     <origin xyz="-0.020233 0.090577 0.013" rpy="0 0 0"/>
     <geometry>
-      <mesh filename="package://nhk2026_sim/meshes/alm_1_v4_2.stl" scale="0.001 0.001 0.001"/>
+      <mesh filename="file://$(find nhk2026_sim)/meshes/alm_1_v4_2.stl" scale="0.001 0.001 0.001"/>
     </geometry>
   </collision>
@@ -133,5 +133,5 @@
     <origin xyz="0.08369 -0.029423 0.013" rpy="0 0 0"/>
     <geometry>
-      <mesh filename="package://nhk2026_sim/meshes/chassis_unit_v18_3.stl" scale="0.001 0.001 0.001"/>
+      <mesh filename="file://$(find nhk2026_sim)/meshes/chassis_unit_v18_3.stl" scale="0.001 0.001 0.001"/>
     </geometry>
     <material name="steel_satin"/>
@@ -140,5 +140,5 @@
     <origin xyz="0.08369 -0.029423 0.013" rpy="0 0 0"/>
     <geometry>
-      <mesh filename="package://nhk2026_sim/meshes/chassis_unit_v18_3.stl" scale="0.001 0.001 0.001"/>
+      <mesh filename="file://$(find nhk2026_sim)/meshes/chassis_unit_v18_3.stl" scale="0.001 0.001 0.001"/>
     </geometry>
   </collision>
@@ -153,5 +153,5 @@
     <origin xyz="-0.072195 0.023977 0.013" rpy="0 0 0"/>
     <geometry>
-      <mesh filename="package://nhk2026_sim/meshes/LD19_with_mounter_v17_1.stl" scale="0.001 0.001 0.001"/>
+      <mesh filename="file://$(find nhk2026_sim)/meshes/LD19_with_mounter_v17_1.stl" scale="0.001 0.001 0.001"/>
     </geometry>
     <material name="steel_satin"/>
@@ -160,5 +160,5 @@
     <origin xyz="-0.072195 0.023977 0.013" rpy="0 0 0"/>
     <geometry>
-      <mesh filename="package://nhk2026_sim/meshes/LD19_with_mounter_v17_1.stl" scale="0.001 0.001 0.001"/>
+      <mesh filename="file://$(find nhk2026_sim)/meshes/LD19_with_mounter_v17_1.stl" scale="0.001 0.001 0.001"/>
     </geometry>
   </collision>
@@ -173,5 +173,5 @@
     <origin xyz="0.044719 0.053077 0.013" rpy="0 0 0"/>
     <geometry>
-      <mesh filename="package://nhk2026_sim/meshes/fun_adapter_v2_1.stl" scale="0.001 0.001 0.001"/>
+      <mesh filename="file://$(find nhk2026_sim)/meshes/fun_adapter_v2_1.stl" scale="0.001 0.001 0.001"/>
     </geometry>
     <material name="steel_satin"/>
@@ -180,5 +180,5 @@
     <origin xyz="0.044719 0.053077 0.013" rpy="0 0 0"/>
     <geometry>
-      <mesh filename="package://nhk2026_sim/meshes/fun_adapter_v2_1.stl" scale="0.001 0.001 0.001"/>
+      <mesh filename="file://$(find nhk2026_sim)/meshes/fun_adapter_v2_1.stl" scale="0.001 0.001 0.001"/>
     </geometry>
   </collision>
@@ -193,5 +193,5 @@
     <origin xyz="0.065593 0.061233 0.016" rpy="0 0 0"/>
     <geometry>
-      <mesh filename="package://nhk2026_sim/meshes/fun_v13_1.stl" scale="0.001 0.001 0.001"/>
+      <mesh filename="file://$(find nhk2026_sim)/meshes/fun_v13_1.stl" scale="0.001 0.001 0.001"/>
     </geometry>
     <material name="steel_satin"/>
@@ -200,5 +200,5 @@
     <origin xyz="0.065593 0.061233 0.016" rpy="0 0 0"/>
     <geometry>
-      <mesh filename="package://nhk2026_sim/meshes/fun_v13_1.stl" scale="0.001 0.001 0.001"/>
+      <mesh filename="file://$(find nhk2026_sim)/meshes/fun_v13_1.stl" scale="0.001 0.001 0.001"/>
     </geometry>
   </collision>
