Commit message: r2_step_climberのURDFおよびXACROファイルのパッケージ参照を修正し、nhk2026_simに統一

File: src/nhk2026_sim/urdf/r2_step_climber.xacro (robot description, xacro)
@@ -1,6 +1,6 @@
 <?xml version="1.0" ?>
 <robot name="r2_step_climber" xmlns:xacro="http://www.ros.org/wiki/xacro">
-<xacro:include filename="$(find r2_step_climber_description)/urdf/materials.xacro" />
-<xacro:include filename="$(find r2_step_climber_description)/urdf/r2_step_climber.trans" />
+<xacro:include filename="$(find nhk2026_sim)/urdf/materials.xacro" />
+<xacro:include filename="$(find nhk2026_sim)/urdf/r2_step_climber.trans" />
 <link name="base_root_r2"/>
 <link name="base_link_r2">
@@ -13,5 +13,5 @@
     <origin xyz="0 0 0" rpy="0 0 0"/>
     <geometry>
-      <mesh filename="package://r2_step_climber_description/meshes/base_link_r2.stl" scale="0.001 0.001 0.001"/>
+      <mesh filename="package://nhk2026_sim/meshes/base_link_r2.stl" scale="0.001 0.001 0.001"/>
     </geometry>
     <material name="aluminum_satin"/>
@@ -20,5 +20,5 @@
     <origin xyz="0 0 0" rpy="0 0 0"/>
     <geometry>
-      <mesh filename="package://r2_step_climber_description/meshes/base_link_r2.stl" scale="0.001 0.001 0.001"/>
+      <mesh filename="package://nhk2026_sim/meshes/base_link_r2.stl" scale="0.001 0.001 0.001"/>
     </geometry>
   </collision>
@@ -33,5 +33,5 @@
     <origin xyz="-0.019 0.31 -0.06" rpy="0 0 0"/>
     <geometry>
-      <mesh filename="package://r2_step_climber_description/meshes/R2_step_clibmer_arm_v2_1.stl" scale="0.001 0.001 0.001"/>
+      <mesh filename="package://nhk2026_sim/meshes/R2_step_clibmer_arm_v2_1.stl" scale="0.001 0.001 0.001"/>
     </geometry>
     <material name="aluminum_satin"/>
@@ -40,5 +40,5 @@
     <origin xyz="-0.019 0.31 -0.06" rpy="0 0 0"/>
     <geometry>
-      <mesh filename="package://r2_step_climber_description/meshes/R2_step_clibmer_arm_v2_1.stl" scale="0.001 0.001 0.001"/>
+      <mesh filename="package://nhk2026_sim/meshes/R2_step_clibmer_arm_v2_1.stl" scale="0.001 0.001 0.001"/>
     </geometry>
   </collision>
@@ -53,5 +53,5 @@
     <origin xyz="0.275 -0.095 -0.06" rpy="0 0 0"/>
     <geometry>
-      <mesh filename="package://r2_step_climber_description/meshes/R2_step_climber_front_v2_1.stl" scale="0.001 0.001 0.001"/>
+      <mesh filename="package://nhk2026_sim/meshes/R2_step_climber_front_v2_1.stl" scale="0.001 0.001 0.001"/>
     </geometry>
     <material name="aluminum_satin"/>
@@ -60,5 +60,5 @@
     <origin xyz="0.275 -0.095 -0.06" rpy="0 0 0"/>
     <geometry>
-      <mesh filename="package://r2_step_climber_description/meshes/R2_step_climber_front_v2_1.stl" scale="0.001 0.001 0.001"/>
+      <mesh filename="package://nhk2026_sim/meshes/R2_step_climber_front_v2_1.stl" scale="0.001 0.001 0.001"/>
     </geometry>
   </collision>
@@ -73,5 +73,5 @@
     <origin xyz="-0.275 -0.095 -0.06" rpy="0 0 0"/>
     <geometry>
-      <mesh filename="package://r2_step_climber_description/meshes/R2_step_climber_front_v2_2.stl" scale="0.001 0.001 0.001"/>
+      <mesh filename="package://nhk2026_sim/meshes/R2_step_climber_front_v2_2.stl" scale="0.001 0.001 0.001"/>
     </geometry>
     <material name="aluminum_satin"/>
@@ -80,5 +80,5 @@
     <origin xyz="-0.275 -0.095 -0.06" rpy="0 0 0"/>
     <geometry>
-      <mesh filename="package://r2_step_climber_description/meshes/R2_step_climber_front_v2_2.stl" scale="0.001 0.001 0.001"/>
+      <mesh filename="package://nhk2026_sim/meshes/R2_step_climber_front_v2_2.stl" scale="0.001 0.001 0.001"/>
     </geometry>
   </collision>
