Commit message: LIDARセンサー用のリンクとジョイントを追加

File: src/nhk2026_sim/urdf/r2_robot.xacro (robot description, xacro)
@@ -29,3 +29,15 @@
   </collision>
 </link>
+<link name="lidar_front"/>
+<link name="lidar_back"/>
+<joint name="base_link_to_lidar_front" type="fixed">
+  <origin xyz="-0.094036 0.2255 0.0755" rpy="0 0 1.5707"/>
+  <parent link="base_link"/>
+  <child link="lidar_front"/>
+</joint>
+<joint name="base_link_to_lidar_back" type="fixed">
+  <origin xyz="0.2084 -0.2999 0.0755" rpy="0 0 0"/>
+  <parent link="base_link"/>
+  <child link="lidar_back"/>
+</joint>
 </robot>

Commit message: R2ロボットのURDFとシミュレーション環境を更新し、センサー設定を改善

File: src/nhk2026_sim/urdf/r2_robot.xacro (robot description, xacro)
@@ -29,4 +29,10 @@
   </collision>
 </link>
+<link name="base_footprint"/>
+<joint name="base_link_to_base_footprint" type="fixed">
+  <origin xyz="0 0 0" rpy="0 0 0"/>
+  <parent link="base_link"/>
+  <child link="base_footprint"/>
+</joint>
 <link name="lidar_front"/>
 <link name="lidar_back"/>
@@ -49,6 +55,6 @@
         name="ignition::gazebo::systems::OdometryPublisher">
   <odom_frame>odom</odom_frame>
-  <robot_base_frame>base_footprint</robot_base_frame>
-  <odom_publish_frequency>10</odom_publish_frequency>
+  <robot_base_frame>base_root</robot_base_frame>
+  <odom_publish_frequency>40</odom_publish_frequency>
   <odom_topic>/odom</odom_topic>
   <tf_topic>/tf</tf_topic>
@@ -85,7 +91,4 @@
       </range>
     </ray>
-    <plugin filename="libignition-gazebo-sensors-system.so" name="ignition::gazebo::systems::Sensors">
-        <render_engine>ogre</render_engine>
-    </plugin>
   </sensor>
 </gazebo>
@@ -118,7 +121,4 @@
       </range>
     </ray>
-    <plugin filename="libignition-gazebo-sensors-system.so" name="ignition::gazebo::systems::Sensors">
-        <render_engine>ogre</render_engine>
-    </plugin>
   </sensor>
 </gazebo>

Commit message: r2 urdf fix

File: src/nhk2026_sim/urdf/r2_robot.xacro (robot description, xacro)
@@ -1,94 +1,88 @@
 <?xml version="1.0" ?>
 <robot name="r2_robot" xmlns:xacro="http://www.ros.org/wiki/xacro">
-<xacro:include filename="$(find nhk2026_sim)/urdf/materials.xacro" />
-<xacro:include filename="$(find nhk2026_sim)/urdf/r2_robot.trans" />
-<link name="base_root"/>
-<joint name="base_root_to_base_link" type="fixed">
-  <origin xyz="0 0 0" rpy="0 0 0"/>
-  <parent link="base_root"/>
-  <child link="base_link"/>
-</joint>
-<link name="base_link">
-  <inertial>
-    <origin xyz="0.06030185659270798 0.06561514891160666 0.304245696022597" rpy="0 0 0"/>
-    <mass value="1032.9670991741832"/>
-    <inertia ixx="58.654004" iyy="37.606623" izz="56.51615" ixy="-6.107741" iyz="11.174448" ixz="6.412628"/>
-  </inertial>
-  <visual>
+  <xacro:include filename="$(find nhk2026_sim)/urdf/materials.xacro" />
+  <xacro:include filename="$(find nhk2026_sim)/urdf/r2_robot.trans" />
+  <link name="base_footprint"/>
+  <link name="base_link">
+    <inertial>
+      <origin xyz="0.06030185659270798 0.06561514891160666 0.304245696022597" rpy="0 0 0"/>
+      <mass value="1032.9670991741832"/>
+      <inertia ixx="58.654004" iyy="37.606623" izz="56.51615" ixy="-6.107741" iyz="11.174448" ixz="6.412628"/>
+    </inertial>
+    <visual>
+      <origin xyz="0 0 0" rpy="0 0 0"/>
+      <geometry>
+        <mesh filename="package://nhk2026_sim/meshes/base_link_r2.stl" scale="0.001 0.001 0.001"/>
+      </geometry>
+      <material name="silicone_white"/>
+    </visual>
+    <collision>
+      <origin xyz="0 0 0" rpy="0 0 0"/>
+      <geometry>
+        <mesh filename="package://nhk2026_sim/meshes/base_link_r2.stl" scale="0.001 0.001 0.001"/>
+      </geometry>
+    </collision>
+  </link>
+  <joint name="base_footprint_to_base_link" type="fixed">
     <origin xyz="0 0 0" rpy="0 0 0"/>
-    <geometry>
-      <mesh filename="package://nhk2026_sim/meshes/base_link_r2.stl" scale="0.001 0.001 0.001"/>
-    </geometry>
-    <material name="silicone_white"/>
-  </visual>
-  <collision>
-    <origin xyz="0 0 0" rpy="0 0 0"/>
-    <geometry>
-      <mesh filename="package://nhk2026_sim/meshes/base_link_r2.stl" scale="0.001 0.001 0.001"/>
-    </geometry>
-  </collision>
-</link>
-<link name="base_footprint"/>
-<joint name="base_link_to_base_footprint" type="fixed">
-  <origin xyz="0 0 0" rpy="0 0 0"/>
-  <parent link="base_link"/>
-  <child link="base_footprint"/>
-</joint>
-<link name="lidar_front"/>
-<link name="lidar_back"/>
-<joint name="base_link_to_lidar_front" type="fixed">
-  <origin xyz="-0.094036 0.2255 0.0755" rpy="0 0 1.5707"/>
-  <parent link="base_link"/>
-  <child link="lidar_front"/>
-</joint>
-<joint name="base_link_to_lidar_back" type="fixed">
-  <origin xyz="0.2084 -0.2999 0.0755" rpy="0 0 0"/>
-  <parent link="base_link"/>
-  <child link="lidar_back"/>
-</joint>
-<gazebo>
-  <plugin filename="libignition-gazebo-velocity-control-system.so"
-          name="ignition::gazebo::systems::VelocityControl">
-    <topic>/cmd_vel</topic>
-  </plugin>
-  <plugin filename="libignition-gazebo-odometry-publisher-system.so"
-        name="ignition::gazebo::systems::OdometryPublisher">
-  <odom_frame>odom</odom_frame>
-  <robot_base_frame>base_root</robot_base_frame>
-  <odom_publish_frequency>40</odom_publish_frequency>
-  <odom_topic>/odom</odom_topic>
-  <tf_topic>/tf</tf_topic>
-  <dimensions>2</dimensions>
-  <gaussian_noise>0.0</gaussian_noise>
-  </plugin>
-</gazebo>
-<gazebo reference="lidar_front">
-  <sensor type="gpu_lidar" name="lidar_sensor_front">
-    <ignition_frame_id>lidar_front</ignition_frame_id>
-    <topic>/scan_front</topic>
-    <alwaysOn>1</alwaysOn>
-    <visualize>true</visualize>
-    <update_rate>40</update_rate>
-    <ray>
-      <scan>
-        <horizontal>
-          <samples>1080</samples>
-          <resolution>1</resolution> <min_angle>-2.35619</min_angle>
-          <max_angle> 2.35619</max_angle>
-        </horizontal>
-        <vertical>
-          <samples>1</samples>
-          <resolution>1</resolution>
-          <min_angle>0.0</min_angle>
-          <max_angle>0.0</max_angle>
-        </vertical>
-      </scan>
-      <range>
-        <min>0.1</min>
-        <max>30.0</max>
-        <resolution>0.001</resolution>
-      </range>
-    </ray>
-  </sensor>
-</gazebo>
+    <parent link="base_footprint"/>
+    <child link="base_link"/>
+  </joint>
+  <link name="lidar_front"/>
+  <link name="lidar_back"/>
+  <joint name="base_link_to_lidar_front" type="fixed">
+    <origin xyz="-0.094036 0.2255 0.0755" rpy="0 0 1.5707"/>
+    <parent link="base_link"/>
+    <child link="lidar_front"/>
+  </joint>
+  <joint name="base_link_to_lidar_back" type="fixed">
+    <origin xyz="0.2084 -0.2999 0.0755" rpy="0 0 0"/>
+    <parent link="base_link"/>
+    <child link="lidar_back"/>
+  </joint>
+  <gazebo>
+    <plugin filename="libignition-gazebo-velocity-control-system.so"
+            name="ignition::gazebo::systems::VelocityControl">
+      <topic>/cmd_vel</topic>
+    </plugin>
+    <plugin filename="libignition-gazebo-odometry-publisher-system.so"
+          name="ignition::gazebo::systems::OdometryPublisher">
+      <odom_frame>odom</odom_frame>
+      <robot_base_frame>base_footprint</robot_base_frame>
+      <odom_publish_frequency>40</odom_publish_frequency>
+      <odom_topic>/odom</odom_topic>
+      <tf_topic>/tf</tf_topic>
+      <dimensions>2</dimensions>
+      <gaussian_noise>0.0</gaussian_noise>
+    </plugin>
+  </gazebo>
+  <gazebo reference="lidar_front">
+    <sensor type="gpu_lidar" name="lidar_sensor_front">
+      <ignition_frame_id>lidar_front</ignition_frame_id>
+      <topic>/scan_front</topic>
+      <alwaysOn>1</alwaysOn>
+      <visualize>true</visualize>
+      <update_rate>40</update_rate>
+      <ray>
+        <scan>
+          <horizontal>
+            <samples>1080</samples>
+            <resolution>1</resolution> <min_angle>-2.35619</min_angle>
+            <max_angle> 2.35619</max_angle>
+          </horizontal>
+          <vertical>
+            <samples>1</samples>
+            <resolution>1</resolution>
+            <min_angle>0.0</min_angle>
+            <max_angle>0.0</max_angle>
+          </vertical>
+        </scan>
+        <range>
+          <min>0.1</min>
+          <max>30.0</max>
+          <resolution>0.001</resolution>
+        </range>
+      </ray>
+    </sensor>
+  </gazebo>
 </robot>

Commit message: mcl tf fix

File: src/nhk2026_sim/urdf/r2_robot.xacro (robot description, xacro)
@@ -25,5 +25,5 @@
   </link>
   <joint name="base_footprint_to_base_link" type="fixed">
-    <origin xyz="0 0 0" rpy="0 0 0"/>
+    <origin xyz="0 0 0.1" rpy="0 0 0"/>
     <parent link="base_footprint"/>
     <child link="base_link"/>

Commit message: tf fix

File: src/nhk2026_sim/urdf/r2_robot.xacro (robot description, xacro)
@@ -25,5 +25,5 @@
   </link>
   <joint name="base_footprint_to_base_link" type="fixed">
-    <origin xyz="0 0 0.1" rpy="0 0 0"/>
+    <origin xyz="0 0 0" rpy="0 0 0"/>
     <parent link="base_footprint"/>
     <child link="base_link"/>

Commit message: sim治ってそう

File: src/nhk2026_sim/urdf/r2_robot.xacro (robot description, xacro)
@@ -6,7 +6,7 @@
   <link name="base_link">
     <inertial>
-      <origin xyz="0.06030185659270798 0.06561514891160666 0.304245696022597" rpy="0 0 0"/>
-      <mass value="1032.9670991741832"/>
-      <inertia ixx="58.654004" iyy="37.606623" izz="56.51615" ixy="-6.107741" iyz="11.174448" ixz="6.412628"/>
+      <origin xyz="0 0 0.1" rpy="0 0 0"/>
+      <mass value="20.0"/>
+      <inertia ixx="0.48" iyy="0.48" izz="0.83" ixy="0" iyz="0" ixz="0"/>
     </inertial>
     <visual>

Commit message: urdf change

File: src/nhk2026_sim/urdf/r2_robot.xacro (robot description, xacro)
@@ -32,5 +32,5 @@
   <link name="lidar_back"/>
   <joint name="base_link_to_lidar_front" type="fixed">
-    <origin xyz="-0.094036 0.2255 0.0755" rpy="0 0 1.5707"/>
+    <origin xyz="-0.094036 0.2255 0.0755" rpy="3.14159 0 1.5707"/>
     <parent link="base_link"/>
     <child link="lidar_front"/>

Commit message: sim環境は作れた

File: src/nhk2026_sim/urdf/r2_robot.xacro (robot description, xacro)
@@ -123,3 +123,36 @@
     <kd>100.0</kd>
   </gazebo>
+  <link name="livox_frame"/>
+  <joint name="base_link_to_livox" type="fixed">
+    <origin xyz="-0.25 0.30 0.80" rpy="3.14159 0 0"/>
+    <parent link="base_link"/>
+    <child link="livox_frame"/>
+  </joint>
+  <gazebo reference="livox_frame">
+    <sensor type="gpu_lidar" name="livox_mid360_sensor">
+      <ignition_frame_id>livox_frame</ignition_frame_id>
+      <topic>/livox</topic>
+      <alwaysOn>1</alwaysOn>
+      <visualize>true</visualize>
+      <update_rate>10</update_rate> <ray>
+        <scan>
+          <horizontal>
+            <samples>1000</samples>
+            <resolution>1</resolution>
+            <min_angle>-3.14159</min_angle>
+            <max_angle>3.14159</max_angle>
+          </horizontal>
+          <vertical>
+            <samples>64</samples> <resolution>1</resolution>
+            <min_angle>-0.12217</min_angle>
+            <max_angle>0.90757</max_angle>
+          </vertical>
+        </scan>
+        <range>
+          <min>0.1</min>
+          <max>40.0</max> <resolution>0.003</resolution>
+        </range>
+      </ray>
+    </sensor>
+  </gazebo>
 </robot>

Commit message: launch add

File: src/nhk2026_sim/urdf/r2_robot.xacro (robot description, xacro)
@@ -32,10 +32,10 @@
   <link name="lidar_back"/>
   <joint name="base_link_to_lidar_front" type="fixed">
-    <origin xyz="-0.094036 0.2255 0.0755" rpy="3.14159 0 1.5707"/>
+    <origin xyz="-0.157 0.2885 0.0755" rpy="3.14159 0 1.5707"/>
     <parent link="base_link"/>
     <child link="lidar_front"/>
   </joint>
   <joint name="base_link_to_lidar_back" type="fixed">
-    <origin xyz="0.2084 -0.2999 0.0755" rpy="0 0 0"/>
+    <origin xyz="0.270 -0.3615 0.0755" rpy="3.14159 0 0"/>
     <parent link="base_link"/>
     <child link="lidar_back"/>
@@ -125,5 +125,5 @@
   <link name="livox_frame"/>
   <joint name="base_link_to_livox" type="fixed">
-    <origin xyz="-0.25 0.30 0.80" rpy="3.14159 0 0"/>
+    <origin xyz="-0.325 -0.03 0.382" rpy="3.14159 0 0"/>
     <parent link="base_link"/>
     <child link="livox_frame"/>

Commit message: fix

File: src/nhk2026_sim/urdf/r2_robot.xacro (robot description, xacro)
@@ -125,5 +125,5 @@
   <link name="livox_frame"/>
   <joint name="base_link_to_livox" type="fixed">
-    <origin xyz="-0.325 -0.03 0.382" rpy="3.14159 0 0"/>
+    <origin xyz="-0.325 -0.03 0.382" rpy="3.14159 1.57 0"/>
     <parent link="base_link"/>
     <child link="livox_frame"/>

Commit message: fix

File: src/nhk2026_sim/urdf/r2_robot.xacro (robot description, xacro)
@@ -125,5 +125,5 @@
   <link name="livox_frame"/>
   <joint name="base_link_to_livox" type="fixed">
-    <origin xyz="-0.325 -0.03 0.382" rpy="3.14159 1.57 0"/>
+    <origin xyz="-0.325 -0.03 0.382" rpy="3.14159 0 1.57"/>
     <parent link="base_link"/>
     <child link="livox_frame"/>

Commit message: fix

File: src/nhk2026_sim/urdf/r2_robot.xacro (robot description, xacro)
@@ -125,5 +125,5 @@
   <link name="livox_frame"/>
   <joint name="base_link_to_livox" type="fixed">
-    <origin xyz="-0.325 -0.03 0.382" rpy="3.14159 0 1.57"/>
+    <origin xyz="-0.325 -0.03 0.382" rpy="3.14159 0 -1.57"/>
     <parent link="base_link"/>
     <child link="livox_frame"/>

Commit message: fix

File: src/nhk2026_sim/urdf/r2_robot.xacro (robot description, xacro)
@@ -125,5 +125,5 @@
   <link name="livox_frame"/>
   <joint name="base_link_to_livox" type="fixed">
-    <origin xyz="-0.325 -0.03 0.382" rpy="3.14159 0 -1.57"/>
+    <origin xyz="-0.325 -0.03 0.443" rpy="3.14159 0 -1.57"/>
     <parent link="base_link"/>
     <child link="livox_frame"/>

Commit message: fix

File: src/nhk2026_sim/urdf/r2_robot.xacro (robot description, xacro)
@@ -125,5 +125,5 @@
   <link name="livox_frame"/>
   <joint name="base_link_to_livox" type="fixed">
-    <origin xyz="-0.325 -0.03 0.443" rpy="3.14159 0 -1.57"/>
+    <origin xyz="-0.325 -0.03 0.423" rpy="3.14159 0 -1.57"/>
     <parent link="base_link"/>
     <child link="livox_frame"/>

Commit message: Revert "Merge pull request #96 from T-semi-Tohoku-Uni/70-livox"
This reverts commit cc21be75c26a1e70e68cb631454f5c229d969a9b, reversing
changes made to 68540fca285e15eb7521a5334f341a0dc6f3f876.

File: src/nhk2026_sim/urdf/r2_robot.xacro (robot description, xacro)
@@ -32,10 +32,10 @@
   <link name="lidar_back"/>
   <joint name="base_link_to_lidar_front" type="fixed">
-    <origin xyz="-0.157 0.2885 0.0755" rpy="3.14159 0 1.5707"/>
+    <origin xyz="-0.094036 0.2255 0.0755" rpy="3.14159 0 1.5707"/>
     <parent link="base_link"/>
     <child link="lidar_front"/>
   </joint>
   <joint name="base_link_to_lidar_back" type="fixed">
-    <origin xyz="0.270 -0.3615 0.0755" rpy="3.14159 0 0"/>
+    <origin xyz="0.2084 -0.2999 0.0755" rpy="0 0 0"/>
     <parent link="base_link"/>
     <child link="lidar_back"/>
@@ -53,5 +53,5 @@
       <odom_topic>/odom</odom_topic>
       <tf_topic>/tf</tf_topic>
-      <dimensions>3</dimensions>
+      <dimensions>2</dimensions>
       <gaussian_noise>0.0</gaussian_noise>
     </plugin>
@@ -123,36 +123,3 @@
     <kd>100.0</kd>
   </gazebo>
-  <link name="livox_frame"/>
-  <joint name="base_link_to_livox" type="fixed">
-    <origin xyz="-0.325 -0.03 0.423" rpy="3.14159 0 -1.57"/>
-    <parent link="base_link"/>
-    <child link="livox_frame"/>
-  </joint>
-  <gazebo reference="livox_frame">
-    <sensor type="gpu_lidar" name="livox_mid360_sensor">
-      <ignition_frame_id>livox_frame</ignition_frame_id>
-      <topic>/livox</topic>
-      <alwaysOn>1</alwaysOn>
-      <visualize>true</visualize>
-      <update_rate>10</update_rate> <ray>
-        <scan>
-          <horizontal>
-            <samples>1000</samples>
-            <resolution>1</resolution>
-            <min_angle>-3.14159</min_angle>
-            <max_angle>3.14159</max_angle>
-          </horizontal>
-          <vertical>
-            <samples>64</samples> <resolution>1</resolution>
-            <min_angle>-0.12217</min_angle>
-            <max_angle>0.90757</max_angle>
-          </vertical>
-        </scan>
-        <range>
-          <min>0.1</min>
-          <max>40.0</max> <resolution>0.003</resolution>
-        </range>
-      </ray>
-    </sensor>
-  </gazebo>
 </robot>
