Commit message: IdeArmActionServerクラスのフィードバックタイマーコールバックにループレートを追加し、launchファイルでjoint_state_publisherをjoint_state_publisher_guiに変更

File: src/nhk2026_sim/urdf/ide_arm.xacro (robot description, xacro)
@@ -103,4 +103,5 @@
   </collision>
 </link>
+<link name="tcp_link"/>
 <joint name="fix" type="fixed">
   <origin xyz="0.0 0.0 0.0" rpy="0 0 0"/>
@@ -126,5 +127,10 @@
   <parent link="link_2_v1_1"/>
   <child link="end_effector_v1_1"/>
-  <axis xyz="-1.0 -0.0 0.0"/>
+  <axis xyz="1.0 0.0 0.0"/>
+</joint>
+<joint name="end_effector" type="fixed">
+  <origin xyz="-0.15 0.230 0" rpy="0 0 0"/>
+  <parent link="end_effector_v1_1"/>
+  <child link="tcp_link"/>
 </joint>
 </robot>

Commit message: base_linkとfixジョイントを削除し、ide_arm.xacroを整理

File: src/nhk2026_sim/urdf/ide_arm.xacro (robot description, xacro)
@@ -3,24 +3,4 @@
 <xacro:include filename="$(find nhk2026_sim)/urdf/materials.xacro" />
 <xacro:include filename="$(find nhk2026_sim)/urdf/ide_arm.trans" />
-<link name="base_link">
-  <inertial>
-    <origin xyz="0.0 0.0 -0.0005" rpy="0 0 0"/>
-    <mass value="0.019624999999999997"/>
-    <inertia ixx="4e-06" iyy="4e-06" izz="8e-06" ixy="0.0" iyz="0.0" ixz="0.0"/>
-  </inertial>
-  <visual>
-    <origin xyz="0 0 0" rpy="0 0 0"/>
-    <geometry>
-      <mesh filename="package://nhk2026_sim/meshes/base_link_ide_arm.stl" scale="1.0 1.0 1.0"/>
-    </geometry>
-    <material name="_"/>
-  </visual>
-  <collision>
-    <origin xyz="0 0 0" rpy="0 0 0"/>
-    <geometry>
-      <mesh filename="package://nhk2026_sim/meshes/base_link_ide_arm.stl" scale="1.0 1.0 1.0"/>
-    </geometry>
-  </collision>
-</link>
 <link name="link_1_v2_1">
   <inertial>
@@ -104,9 +84,4 @@
 </link>
 <link name="tcp_link"/>
-<joint name="fix" type="fixed">
-  <origin xyz="0.0 0.0 0.0" rpy="0 0 0"/>
-  <parent link="base_link"/>
-  <child link="arm_base_v2_1"/>
-</joint>
 <joint name="joint1" type="revolute">
   <origin xyz="-0.005751 0.088 0.13" rpy="0 0 0"/>

Commit message: ide_arm.xacroにarm_baseリンクを追加し、各リンクの材質をaluminum_satinに変更。fixジョイントを追加。

File: src/nhk2026_sim/urdf/ide_arm.xacro (robot description, xacro)
@@ -3,4 +3,5 @@
 <xacro:include filename="$(find nhk2026_sim)/urdf/materials.xacro" />
 <xacro:include filename="$(find nhk2026_sim)/urdf/ide_arm.trans" />
+<link name="arm_base"/>
 <link name="link_1_v2_1">
   <inertial>
@@ -14,5 +15,5 @@
       <mesh filename="package://nhk2026_sim/meshes/link_1_v2_1.stl" scale="1.0 1.0 1.0"/>
     </geometry>
-    <material name="_"/>
+    <material name="aluminum_satin"/>
   </visual>
   <collision>
@@ -34,5 +35,5 @@
       <mesh filename="package://nhk2026_sim/meshes/link_2_v1_1.stl" scale="1.0 1.0 1.0"/>
     </geometry>
-    <material name="_"/>
+    <material name="aluminum_satin"/>
   </visual>
   <collision>
@@ -54,5 +55,5 @@
       <mesh filename="package://nhk2026_sim/meshes/end_effector_v1_1.stl" scale="1.0 1.0 1.0"/>
     </geometry>
-    <material name="_"/>
+    <material name="aluminum_satin"/>
   </visual>
   <collision>
@@ -74,5 +75,5 @@
       <mesh filename="package://nhk2026_sim/meshes/arm_base_v2_1.stl" scale="1.0 1.0 1.0"/>
     </geometry>
-    <material name="_"/>
+    <material name="aluminum_satin"/>
   </visual>
   <collision>
@@ -84,4 +85,8 @@
 </link>
 <link name="tcp_link"/>
+<joint name="fix" type="fixed">
+  <parent link="arm_base"/>
+  <child link="arm_base_v2_1"/>
+</joint>
 <joint name="joint1" type="revolute">
   <origin xyz="-0.005751 0.088 0.13" rpy="0 0 0"/>

Commit message: joint3のオリジンの回転を修正

File: src/nhk2026_sim/urdf/ide_arm.xacro (robot description, xacro)
@@ -104,5 +104,5 @@
 </joint>
 <joint name="joint3" type="continuous">
-  <origin xyz="-0.054 0.1955 0.0572" rpy="0 0 0"/>
+  <origin xyz="-0.054 0.1955 0.0572" rpy="3.141592 0 0"/>
   <parent link="link_2_v1_1"/>
   <child link="end_effector_v1_1"/>

Commit message: joint3のオリジンの回転精度を向上させ、制限を追加

File: src/nhk2026_sim/urdf/ide_arm.xacro (robot description, xacro)
@@ -104,8 +104,9 @@
 </joint>
 <joint name="joint3" type="continuous">
-  <origin xyz="-0.054 0.1955 0.0572" rpy="3.141592 0 0"/>
+  <origin xyz="-0.054 0.1955 0.0572" rpy="3.141593 0 0"/>
   <parent link="link_2_v1_1"/>
   <child link="end_effector_v1_1"/>
   <axis xyz="1.0 0.0 0.0"/>
+  <limit upper="3.141593" lower="-3.141593" effort="100" velocity="100"/>
 </joint>
 <joint name="end_effector" type="fixed">

Commit message: add gazebo plugin

File: src/nhk2026_sim/urdf/ide_arm.xacro (robot description, xacro)
@@ -103,5 +103,5 @@
   <limit upper="0.302" lower="0.0" effort="100" velocity="100"/>
 </joint>
-<joint name="joint3" type="continuous">
+<joint name="joint3" type="revolute">
   <origin xyz="-0.054 0.1955 0.0572" rpy="3.141593 0 0"/>
   <parent link="link_2_v1_1"/>
@@ -115,3 +115,26 @@
   <child link="tcp_link"/>
 </joint>
+<gazebo>
+  <plugin filename="gz-sim-joint-position-controller-system"
+          name="gz::sim::systems::JointPositionController">
+    <joint_name>joint1</joint_name>
+    <joint_index>0</joint_index>
+    <topic>/joint1</topic>
+    <p_gain>5.0</p_gain>
+  </plugin>
+  <plugin filename="gz-sim-joint-position-controller-system"
+          name="gz::sim::systems::JointPositionController2">
+    <joint_name>joint2</joint_name>
+    <joint_index>0</joint_index>
+    <topic>/joint2</topic>
+    <p_gain>5.0</p_gain>
+  </plugin>
+  <plugin filename="gz-sim-joint-position-controller-system"
+          name="gz::sim::systems::JointPositionController3">
+    <joint_name>joint3</joint_name>
+    <joint_index>0</joint_index>
+    <topic>/joint3</topic>
+    <p_gain>5.0</p_gain>
+  </plugin>
+</gazebo>
 </robot>

Commit message: update robot launch and xacro files, add arm_plane world and bridge node for simulation

File: src/nhk2026_sim/urdf/ide_arm.xacro (robot description, xacro)
@@ -116,23 +116,27 @@
 </joint>
 <gazebo>
+  <joint name="arm_base_world_fixed" type="fixed">
+    <parent>world</parent>
+    <child>arm_base</child>
+  </joint>
   <plugin filename="gz-sim-joint-position-controller-system"
           name="gz::sim::systems::JointPositionController">
-    <joint_name>joint_sim1</joint_name>
+    <joint_name>joint1</joint_name>
     <joint_index>0</joint_index>
-    <topic>/joint1</topic>
+    <topic>/joint_sim1</topic>
     <p_gain>5.0</p_gain>
   </plugin>
   <plugin filename="gz-sim-joint-position-controller-system"
-          name="gz::sim::systems::JointPositionController2">
-    <joint_name>joint_sim2</joint_name>
+          name="gz::sim::systems::JointPositionController">
+    <joint_name>joint2</joint_name>
     <joint_index>0</joint_index>
-    <topic>/joint2</topic>
+    <topic>/joint_sim2</topic>
     <p_gain>5.0</p_gain>
   </plugin>
   <plugin filename="gz-sim-joint-position-controller-system"
-          name="gz::sim::systems::JointPositionController3">
-    <joint_name>joint_sim3</joint_name>
+          name="gz::sim::systems::JointPositionController">
+    <joint_name>joint3</joint_name>
     <joint_index>0</joint_index>
-    <topic>/joint3</topic>
+    <topic>/joint_sim3</topic>
     <p_gain>5.0</p_gain>
   </plugin>

Commit message: update joint limits and controller gains for improved simulation performance

File: src/nhk2026_sim/urdf/ide_arm.xacro (robot description, xacro)
@@ -94,5 +94,5 @@
   <child link="link_1_v2_1"/>
   <axis xyz="1.0 0.0 0.0"/>
-  <limit upper="3.141593" lower="0.0" effort="100" velocity="100"/>
+  <limit upper="3.141593" lower="-3.141593" effort="1000" velocity="100"/>
 </joint>
 <joint name="joint2" type="prismatic">
@@ -127,5 +127,5 @@
     <joint_index>0</joint_index>
     <topic>/joint_sim1</topic>
-    <p_gain>5.0</p_gain>
+    <p_gain>50</p_gain>
     <i_gain>0.1</i_gain>
     <d_gain>0.01</d_gain>
@@ -145,5 +145,5 @@
     <joint_index>0</joint_index>
     <topic>/joint_sim3</topic>
-    <p_gain>5.0</p_gain>
+    <p_gain>50</p_gain>
     <i_gain>0.1</i_gain>
     <d_gain>0.01</d_gain>

Commit message: update joint limits and controller gains for improved performance; add logging for joint completion

File: src/nhk2026_sim/urdf/ide_arm.xacro (robot description, xacro)
@@ -94,5 +94,5 @@
   <child link="link_1_v2_1"/>
   <axis xyz="1.0 0.0 0.0"/>
-  <limit upper="3.141593" lower="-3.141593" effort="1000" velocity="100"/>
+  <limit upper="3.141593" lower="0" effort="1000" velocity="100"/>
 </joint>
 <joint name="joint2" type="prismatic">
@@ -101,5 +101,5 @@
   <child link="link_2_v1_1"/>
   <axis xyz="-0.0 1.0 0.0"/>
-  <limit upper="0.302" lower="0.0" effort="100" velocity="100"/>
+  <limit upper="0.302" lower="0.0" effort="1000" velocity="100"/>
 </joint>
 <joint name="joint3" type="revolute">
@@ -128,5 +128,5 @@
     <topic>/joint_sim1</topic>
     <p_gain>35.0</p_gain>
-    <i_gain>0.0</i_gain>
+    <i_gain>1.0</i_gain>
     <d_gain>4.0</d_gain>
   </plugin>
@@ -137,5 +137,5 @@
     <topic>/joint_sim2</topic>
     <p_gain>120.0</p_gain>
-    <i_gain>0.0</i_gain>
+    <i_gain>1.0</i_gain>
     <d_gain>16.0</d_gain>
   </plugin>
@@ -146,5 +146,5 @@
     <topic>/joint_sim3</topic>
     <p_gain>30.0</p_gain>
-    <i_gain>0.0</i_gain>
+    <i_gain>1.0</i_gain>
     <d_gain>4.0</d_gain>
   </plugin>

Commit message: update joint limits and controller gains for improved performance

File: src/nhk2026_sim/urdf/ide_arm.xacro (robot description, xacro)
@@ -94,5 +94,6 @@
   <child link="link_1_v2_1"/>
   <axis xyz="1.0 0.0 0.0"/>
-  <limit upper="3.141593" lower="0" effort="1000" velocity="100"/>
+  <limit upper="3.141593" lower="0" effort="10000" velocity="100"/>
+  <dynamics damping="30.0" friction="0.2"/>
 </joint>
 <joint name="joint2" type="prismatic">
@@ -101,5 +102,6 @@
   <child link="link_2_v1_1"/>
   <axis xyz="-0.0 1.0 0.0"/>
-  <limit upper="0.302" lower="0.0" effort="1000" velocity="100"/>
+  <limit upper="0.302" lower="0.0" effort="10000" velocity="100"/>
+  <dynamics damping="80.0" friction="0.2"/>
 </joint>
 <joint name="joint3" type="revolute">
@@ -108,5 +110,6 @@
   <child link="end_effector_v1_1"/>
   <axis xyz="1.0 0.0 0.0"/>
-  <limit upper="3.141593" lower="-3.141593" effort="100" velocity="100"/>
+  <limit upper="3.141593" lower="-3.141593" effort="10000" velocity="100"/>
+  <dynamics damping="30.0" friction="0.2"/>
 </joint>
 <joint name="end_effector" type="fixed">
@@ -127,7 +130,7 @@
     <joint_index>0</joint_index>
     <topic>/joint_sim1</topic>
-    <p_gain>35.0</p_gain>
-    <i_gain>1.0</i_gain>
-    <d_gain>4.0</d_gain>
+    <p_gain>300.0</p_gain>
+    <i_gain>25.0</i_gain>
+    <d_gain>48.0</d_gain>
   </plugin>
   <plugin filename="gz-sim-joint-position-controller-system"
@@ -136,7 +139,7 @@
     <joint_index>0</joint_index>
     <topic>/joint_sim2</topic>
-    <p_gain>120.0</p_gain>
-    <i_gain>1.0</i_gain>
-    <d_gain>16.0</d_gain>
+    <p_gain>900.0</p_gain>
+    <i_gain>25.0</i_gain>
+    <d_gain>140.0</d_gain>
   </plugin>
   <plugin filename="gz-sim-joint-position-controller-system"
@@ -145,7 +148,7 @@
     <joint_index>0</joint_index>
     <topic>/joint_sim3</topic>
-    <p_gain>30.0</p_gain>
-    <i_gain>1.0</i_gain>
-    <d_gain>4.0</d_gain>
+    <p_gain>300.0</p_gain>
+    <i_gain>25.0</i_gain>
+    <d_gain>42.0</d_gain>
   </plugin>
 </gazebo>

Commit message: fix: increase joint effort limits for improved performance in ide_arm.xacro feat: add dependencies for orocos_kdl and kdl_parser in CMakeLists.txt and package.xml

File: src/nhk2026_sim/urdf/ide_arm.xacro (robot description, xacro)
@@ -94,5 +94,5 @@
   <child link="link_1_v2_1"/>
   <axis xyz="1.0 0.0 0.0"/>
-  <limit upper="3.141593" lower="0" effort="10000" velocity="100"/>
+  <limit upper="3.141593" lower="0" effort="1000000" velocity="100"/>
   <dynamics damping="30.0" friction="0.2"/>
 </joint>
@@ -102,5 +102,5 @@
   <child link="link_2_v1_1"/>
   <axis xyz="-0.0 1.0 0.0"/>
-  <limit upper="0.302" lower="0.0" effort="10000" velocity="100"/>
+  <limit upper="0.302" lower="0.0" effort="1000000" velocity="100"/>
   <dynamics damping="80.0" friction="0.2"/>
 </joint>
@@ -110,5 +110,5 @@
   <child link="end_effector_v1_1"/>
   <axis xyz="1.0 0.0 0.0"/>
-  <limit upper="3.141593" lower="-3.141593" effort="10000" velocity="100"/>
+  <limit upper="3.141593" lower="-3.141593" effort="1000000" velocity="100"/>
   <dynamics damping="30.0" friction="0.2"/>
 </joint>

Commit message: listen_transformメソッドの変換順序を修正し、ide_arm_bt.xmlでmove_armアクションのyおよびz座標を更新

File: src/nhk2026_sim/urdf/ide_arm.xacro (robot description, xacro)
@@ -110,5 +110,5 @@
   <child link="end_effector_v1_1"/>
   <axis xyz="1.0 0.0 0.0"/>
-  <limit upper="3.141593" lower="-3.141593" effort="1000000" velocity="100"/>
+  <limit upper="3.5" lower="-3.5" effort="1000000" velocity="100"/>
   <dynamics damping="30.0" friction="0.2"/>
 </joint>

Commit message: end_effector_v5.stlを追加し、ide_arm.xacroでのメッシュと位置を更新

File: src/nhk2026_sim/urdf/ide_arm.xacro (robot description, xacro)
@@ -51,14 +51,14 @@
   </inertial>
   <visual>
-    <origin xyz="0.032751 -0.722789 -0.147378" rpy="0 0 0"/>
+    <origin xyz="-0.02 -0.02 -0.005" rpy="0 0 0"/>
     <geometry>
-      <mesh filename="package://nhk2026_sim/meshes/end_effector_v1_1.stl" scale="1.0 1.0 1.0"/>
+      <mesh filename="package://nhk2026_sim/meshes/end_effector_v5.stl" scale="1.0 1.0 1.0"/>
     </geometry>
     <material name="aluminum_satin"/>
   </visual>
   <collision>
-    <origin xyz="0.032751 -0.722789 -0.147378" rpy="0 0 0"/>
+    <origin xyz="-0.02 -0.02 -0.005" rpy="0 0 0"/>
     <geometry>
-      <mesh filename="package://nhk2026_sim/meshes/end_effector_v1_1.stl" scale="1.0 1.0 1.0"/>
+      <mesh filename="package://nhk2026_sim/meshes/end_effector_v5.stl" scale="1.0 1.0 1.0"/>
     </geometry>
   </collision>
@@ -114,5 +114,5 @@
 </joint>
 <joint name="end_effector" type="fixed">
-  <origin xyz="-0.15 0.230 0" rpy="0 0 0"/>
+  <origin xyz="-0.15 0.150 0" rpy="0 0 0"/>
   <parent link="end_effector_v1_1"/>
   <child link="tcp_link"/>
