Commit message: r2_2nd.launch.pyのr2_2nd.xacroをr2_all.xacroに変更; ide_arm_macro.xacroとr2_2nd_macro.xacroを新規作成し、r2_all.xacroで両方のモデルを統合

File: src/nhk2026_sim/urdf/ide_arm.xacro (robot description, xacro)
@@ -2,154 +2,5 @@
 <robot name="ide_arm" xmlns:xacro="http://www.ros.org/wiki/xacro">
 <xacro:include filename="$(find nhk2026_sim)/urdf/materials.xacro" />
-<xacro:include filename="$(find nhk2026_sim)/urdf/ide_arm.trans" />
-<link name="arm_base"/>
-<link name="link_1_v2_1">
-  <inertial>
-    <origin xyz="0.017436936078169506 0.19863903889518106 -0.005800117560290835" rpy="0 0 0"/>
-    <mass value="3.5325291043519966"/>
-    <inertia ixx="0.193016" iyy="0.011365" izz="0.184162" ixy="-0.001521" iyz="-0.002565" ixz="-0.000119"/>
-  </inertial>
-  <visual>
-    <origin xyz="0.005751 -0.088 -0.13" rpy="0 0 0"/>
-    <geometry>
-      <mesh filename="package://nhk2026_sim/meshes/link_1_v2_1.stl" scale="1.0 1.0 1.0"/>
-    </geometry>
-    <material name="aluminum_satin"/>
-  </visual>
-  <collision>
-    <origin xyz="0.005751 -0.088 -0.13" rpy="0 0 0"/>
-    <geometry>
-      <mesh filename="package://nhk2026_sim/meshes/link_1_v2_1.stl" scale="1.0 1.0 1.0"/>
-    </geometry>
-  </collision>
-</link>
-<link name="link_2_v1_1">
-  <inertial>
-    <origin xyz="-0.023583323602407703 0.0881743103170528 0.04123693865974003" rpy="0 0 0"/>
-    <mass value="1.5772939629978953"/>
-    <inertia ixx="0.043814" iyy="0.000956" izz="0.043605" ixy="0.002284" iyz="-0.001987" ixz="0.000231"/>
-  </inertial>
-  <visual>
-    <origin xyz="-0.021249 -0.527289 -0.090178" rpy="0 0 0"/>
-    <geometry>
-      <mesh filename="package://nhk2026_sim/meshes/link_2_v1_1.stl" scale="1.0 1.0 1.0"/>
-    </geometry>
-    <material name="aluminum_satin"/>
-  </visual>
-  <collision>
-    <origin xyz="-0.021249 -0.527289 -0.090178" rpy="0 0 0"/>
-    <geometry>
-      <mesh filename="package://nhk2026_sim/meshes/link_2_v1_1.stl" scale="1.0 1.0 1.0"/>
-    </geometry>
-  </collision>
-</link>
-<link name="end_effector_v1_1">
-  <inertial>
-    <origin xyz="-0.07222853245081884 0.1407827459051364 4.278768657439702e-07" rpy="0 0 0"/>
-    <mass value="0.32794468549770983"/>
-    <inertia ixx="0.003366" iyy="0.00235" izz="0.005662" ixy="0.001697" iyz="-0.0" ixz="-0.0"/>
-  </inertial>
-  <visual>
-    <origin xyz="-0.02 -0.02 -0.005" rpy="0 0 0"/>
-    <geometry>
-      <mesh filename="package://nhk2026_sim/meshes/end_effector_v5.stl" scale="1.0 1.0 1.0"/>
-    </geometry>
-    <material name="aluminum_satin"/>
-  </visual>
-  <collision>
-    <origin xyz="-0.02 -0.02 -0.005" rpy="0 0 0"/>
-    <geometry>
-      <mesh filename="package://nhk2026_sim/meshes/end_effector_v5.stl" scale="1.0 1.0 1.0"/>
-    </geometry>
-  </collision>
-</link>
-<link name="arm_base_v2_1">
-  <inertial>
-    <origin xyz="-0.002721948795508748 0.09113126713684143 0.11794174723065468" rpy="0 0 0"/>
-    <mass value="5.012895745680244"/>
-    <inertia ixx="0.024327" iyy="0.014645" izz="0.015421" ixy="-0.000185" iyz="0.001647" ixz="0.000104"/>
-  </inertial>
-  <visual>
-    <origin xyz="-0.0 -0.0 -0.0" rpy="0 0 0"/>
-    <geometry>
-      <mesh filename="package://nhk2026_sim/meshes/arm_base_v2_1.stl" scale="1.0 1.0 1.0"/>
-    </geometry>
-    <material name="aluminum_satin"/>
-  </visual>
-  <collision>
-    <origin xyz="-0.0 -0.0 -0.0" rpy="0 0 0"/>
-    <geometry>
-      <mesh filename="package://nhk2026_sim/meshes/arm_base_v2_1.stl" scale="1.0 1.0 1.0"/>
-    </geometry>
-  </collision>
-</link>
-<link name="tcp_link"/>
-<joint name="fix" type="fixed">
-  <parent link="arm_base"/>
-  <child link="arm_base_v2_1"/>
-</joint>
-<joint name="joint1" type="revolute">
-  <origin xyz="-0.005751 0.088 0.13" rpy="0 0 0"/>
-  <parent link="arm_base_v2_1"/>
-  <child link="link_1_v2_1"/>
-  <axis xyz="1.0 0.0 0.0"/>
-  <limit upper="3.141593" lower="0" effort="1000000" velocity="100"/>
-  <dynamics damping="30.0" friction="0.2"/>
-</joint>
-<joint name="joint2" type="prismatic">
-  <origin xyz="0.027 0.439289 -0.039822" rpy="0 0 0"/>
-  <parent link="link_1_v2_1"/>
-  <child link="link_2_v1_1"/>
-  <axis xyz="-0.0 1.0 0.0"/>
-  <limit upper="0.302" lower="0.0" effort="1000000" velocity="100"/>
-  <dynamics damping="80.0" friction="0.2"/>
-</joint>
-<joint name="joint3" type="revolute">
-  <origin xyz="-0.054 0.1955 0.0572" rpy="3.141593 0 0"/>
-  <parent link="link_2_v1_1"/>
-  <child link="end_effector_v1_1"/>
-  <axis xyz="1.0 0.0 0.0"/>
-  <limit upper="3.5" lower="-3.5" effort="1000000" velocity="100"/>
-  <dynamics damping="30.0" friction="0.2"/>
-</joint>
-<joint name="end_effector" type="fixed">
-  <origin xyz="-0.15 0.150 0" rpy="0 0 0"/>
-  <parent link="end_effector_v1_1"/>
-  <child link="tcp_link"/>
-</joint>
-<gazebo>
-  <joint name="arm_base_world_fixed" type="fixed">
-    <parent>world</parent>
-    <child>arm_base</child>
-  </joint>
-  <plugin filename="gz-sim-joint-state-publisher-system"
-          name="gz::sim::systems::JointStatePublisher" />
-  <plugin filename="gz-sim-joint-position-controller-system"
-          name="gz::sim::systems::JointPositionController">
-    <joint_name>joint1</joint_name>
-    <joint_index>0</joint_index>
-    <topic>/joint_sim1</topic>
-    <p_gain>900.0</p_gain>
-    <i_gain>25.0</i_gain>
-    <d_gain>48.0</d_gain>
-  </plugin>
-  <plugin filename="gz-sim-joint-position-controller-system"
-          name="gz::sim::systems::JointPositionController">
-    <joint_name>joint2</joint_name>
-    <joint_index>0</joint_index>
-    <topic>/joint_sim2</topic>
-    <p_gain>900.0</p_gain>
-    <i_gain>25.0</i_gain>
-    <d_gain>140.0</d_gain>
-  </plugin>
-  <plugin filename="gz-sim-joint-position-controller-system"
-          name="gz::sim::systems::JointPositionController">
-    <joint_name>joint3</joint_name>
-    <joint_index>0</joint_index>
-    <topic>/joint_sim3</topic>
-    <p_gain>900.0</p_gain>
-    <i_gain>25.0</i_gain>
-    <d_gain>48.0</d_gain>
-  </plugin>
-</gazebo>
+<xacro:include filename="$(find nhk2026_sim)/urdf/ide_arm_macro.xacro" />
+<xacro:ide_arm prefix="" />
 </robot>

File: src/nhk2026_sim/urdf/r2_2nd.xacro (robot description, xacro)
@@ -2,103 +2,5 @@
 <robot name="r2_2nd" xmlns:xacro="http://www.ros.org/wiki/xacro">
 <xacro:include filename="$(find nhk2026_sim)/urdf/materials.xacro" />
-<xacro:include filename="$(find nhk2026_sim)/urdf/r2_2nd.trans" />
-<link name="base_link">
-  <inertial>
-    <origin xyz="-0.01897592062348662 -0.10555425475997327 0.14298974134420891" rpy="0 0 0"/>
-    <mass value="13.072259884111979"/>
-    <inertia ixx="1.047084" iyy="1.016092" izz="1.499027" ixy="0.043842" iyz="0.037546" ixz="0.102502"/>
-  </inertial>
-  <visual>
-    <origin xyz="0 0 0" rpy="0 0 0"/>
-    <geometry>
-      <mesh filename="package://nhk2026_sim/meshes/base_link_r2.stl" scale="0.001 0.001 0.001"/>
-    </geometry>
-    <material name="steel_satin"/>
-  </visual>
-  <collision>
-    <origin xyz="0 0 0" rpy="0 0 0"/>
-    <geometry>
-      <mesh filename="package://nhk2026_sim/meshes/base_link_r2.stl" scale="0.001 0.001 0.001"/>
-    </geometry>
-  </collision>
-</link>
-<link name="R2_step_climber_front_v2_1">
-  <inertial>
-    <origin xyz="0.016127121216774898 0.18644792175710703 -2.1817373602184276e-10" rpy="0 0 0"/>
-    <mass value="1.2591666960686572"/>
-    <inertia ixx="0.007687" iyy="0.000408" izz="0.007414" ixy="-8.7e-05" iyz="0.0" ixz="0.0"/>
-  </inertial>
-  <visual>
-    <origin xyz="-0.335 -0.095 -0.06" rpy="0 0 0"/>
-    <geometry>
-      <mesh filename="package://nhk2026_sim/meshes/R2_step_climber_front_v2_1.stl" scale="0.001 0.001 0.001"/>
-    </geometry>
-    <material name="steel_satin"/>
-  </visual>
-  <collision>
-    <origin xyz="-0.335 -0.095 -0.06" rpy="0 0 0"/>
-    <geometry>
-      <mesh filename="package://nhk2026_sim/meshes/R2_step_climber_front_v2_1.stl" scale="0.001 0.001 0.001"/>
-    </geometry>
-  </collision>
-</link>
-<link name="R2_step_climber_front_v2_2">
-  <inertial>
-    <origin xyz="-0.016127121215468332 -0.18644792175710334 -2.1817370132737324e-10" rpy="0 0 0"/>
-    <mass value="1.2591666960686572"/>
-    <inertia ixx="0.007687" iyy="0.000408" izz="0.007414" ixy="-8.7e-05" iyz="-0.0" ixz="-0.0"/>
-  </inertial>
-  <visual>
-    <origin xyz="0.335 -0.095 -0.06" rpy="0 0 0"/>
-    <geometry>
-      <mesh filename="package://nhk2026_sim/meshes/R2_step_climber_front_v2_2.stl" scale="0.001 0.001 0.001"/>
-    </geometry>
-    <material name="steel_satin"/>
-  </visual>
-  <collision>
-    <origin xyz="0.335 -0.095 -0.06" rpy="0 0 0"/>
-    <geometry>
-      <mesh filename="package://nhk2026_sim/meshes/R2_step_climber_front_v2_2.stl" scale="0.001 0.001 0.001"/>
-    </geometry>
-  </collision>
-</link>
-<link name="R2_step_clibmer_arm_v2_1">
-  <inertial>
-    <origin xyz="-0.008920789398712332 0.004691281182066187 0.20281005076730813" rpy="0 0 0"/>
-    <mass value="2.376029715091139"/>
-    <inertia ixx="0.011384" iyy="0.031797" izz="0.022759" ixy="2.2e-05" iyz="0.000365" ixz="-0.000359"/>
-  </inertial>
-  <visual>
-    <origin xyz="-0.019 0.37 -0.06" rpy="0 0 0"/>
-    <geometry>
-      <mesh filename="package://nhk2026_sim/meshes/R2_step_clibmer_arm_v2_1.stl" scale="0.001 0.001 0.001"/>
-    </geometry>
-    <material name="steel_satin"/>
-  </visual>
-  <collision>
-    <origin xyz="-0.019 0.37 -0.06" rpy="0 0 0"/>
-    <geometry>
-      <mesh filename="package://nhk2026_sim/meshes/R2_step_clibmer_arm_v2_1.stl" scale="0.001 0.001 0.001"/>
-    </geometry>
-  </collision>
-</link>
-<joint name="right" type="continuous">
-  <origin xyz="0.335 0.095 0.06" rpy="0 0 0"/>
-  <parent link="base_link"/>
-  <child link="R2_step_climber_front_v2_1"/>
-  <axis xyz="1.0 0.0 0.0"/>
-</joint>
-<joint name="left" type="continuous">
-  <origin xyz="-0.335 0.095 0.06" rpy="0 0 0"/>
-  <parent link="base_link"/>
-  <child link="R2_step_climber_front_v2_2"/>
-  <axis xyz="-1.0 0.0 0.0"/>
-</joint>
-<joint name="back" type="revolute">
-  <origin xyz="0.019 -0.37 0.06" rpy="0 0 0"/>
-  <parent link="base_link"/>
-  <child link="R2_step_clibmer_arm_v2_1"/>
-  <axis xyz="-1.0 0.0 0.0"/>
-  <limit upper="6.283185" lower="3.141593" effort="100" velocity="100"/>
-</joint>
+<xacro:include filename="$(find nhk2026_sim)/urdf/r2_2nd_macro.xacro" />
+<xacro:r2_2nd prefix="" />
 </robot>
