Commit message: launchファイルでjoint_state_publisherを使用するように変更し、URDFモデルのスケールを修正

File: src/ide_arm_description/urdf/ide_arm.xacro (robot description, xacro)
@@ -12,5 +12,5 @@
     <origin xyz="0 0 0" rpy="0 0 0"/>
     <geometry>
-      <mesh filename="package://ide_arm_description/meshes/base_link.stl" scale="0.001 0.001 0.001"/>
+      <mesh filename="package://ide_arm_description/meshes/base_link.stl" scale="1.0 1.0 1.0"/>
     </geometry>
     <material name="_"/>
@@ -19,5 +19,5 @@
     <origin xyz="0 0 0" rpy="0 0 0"/>
     <geometry>
-      <mesh filename="package://ide_arm_description/meshes/base_link.stl" scale="0.001 0.001 0.001"/>
+      <mesh filename="package://ide_arm_description/meshes/base_link.stl" scale="1.0 1.0 1.0"/>
     </geometry>
   </collision>
@@ -32,5 +32,5 @@
     <origin xyz="0.005751 -0.088 -0.13" rpy="0 0 0"/>
     <geometry>
-      <mesh filename="package://ide_arm_description/meshes/link_1_v2_1.stl" scale="0.001 0.001 0.001"/>
+      <mesh filename="package://ide_arm_description/meshes/link_1_v2_1.stl" scale="1.0 1.0 1.0"/>
     </geometry>
     <material name="_"/>
@@ -39,5 +39,5 @@
     <origin xyz="0.005751 -0.088 -0.13" rpy="0 0 0"/>
     <geometry>
-      <mesh filename="package://ide_arm_description/meshes/link_1_v2_1.stl" scale="0.001 0.001 0.001"/>
+      <mesh filename="package://ide_arm_description/meshes/link_1_v2_1.stl" scale="1.0 1.0 1.0"/>
     </geometry>
   </collision>
@@ -52,5 +52,5 @@
     <origin xyz="-0.021249 -0.527289 -0.090178" rpy="0 0 0"/>
     <geometry>
-      <mesh filename="package://ide_arm_description/meshes/link_2_v1_1.stl" scale="0.001 0.001 0.001"/>
+      <mesh filename="package://ide_arm_description/meshes/link_2_v1_1.stl" scale="1.0 1.0 1.0"/>
     </geometry>
     <material name="_"/>
@@ -59,5 +59,5 @@
     <origin xyz="-0.021249 -0.527289 -0.090178" rpy="0 0 0"/>
     <geometry>
-      <mesh filename="package://ide_arm_description/meshes/link_2_v1_1.stl" scale="0.001 0.001 0.001"/>
+      <mesh filename="package://ide_arm_description/meshes/link_2_v1_1.stl" scale="1.0 1.0 1.0"/>
     </geometry>
   </collision>
@@ -72,5 +72,5 @@
     <origin xyz="0.032751 -0.722789 -0.147378" rpy="0 0 0"/>
     <geometry>
-      <mesh filename="package://ide_arm_description/meshes/end_effector_v1_1.stl" scale="0.001 0.001 0.001"/>
+      <mesh filename="package://ide_arm_description/meshes/end_effector_v1_1.stl" scale="1.0 1.0 1.0"/>
     </geometry>
     <material name="_"/>
@@ -79,5 +79,5 @@
     <origin xyz="0.032751 -0.722789 -0.147378" rpy="0 0 0"/>
     <geometry>
-      <mesh filename="package://ide_arm_description/meshes/end_effector_v1_1.stl" scale="0.001 0.001 0.001"/>
+      <mesh filename="package://ide_arm_description/meshes/end_effector_v1_1.stl" scale="1.0 1.0 1.0"/>
     </geometry>
   </collision>
@@ -92,5 +92,5 @@
     <origin xyz="-0.0 -0.0 -0.0" rpy="0 0 0"/>
     <geometry>
-      <mesh filename="package://ide_arm_description/meshes/arm_base_v2_1.stl" scale="0.001 0.001 0.001"/>
+      <mesh filename="package://ide_arm_description/meshes/arm_base_v2_1.stl" scale="1.0 1.0 1.0"/>
     </geometry>
     <material name="_"/>
@@ -99,8 +99,13 @@
     <origin xyz="-0.0 -0.0 -0.0" rpy="0 0 0"/>
     <geometry>
-      <mesh filename="package://ide_arm_description/meshes/arm_base_v2_1.stl" scale="0.001 0.001 0.001"/>
+      <mesh filename="package://ide_arm_description/meshes/arm_base_v2_1.stl" scale="1.0 1.0 1.0"/>
     </geometry>
   </collision>
 </link>
+<joint name="fix" type="fixed">
+  <origin xyz="0.0 0.0 0.0" rpy="0 0 0"/>
+  <parent link="base_link"/>
+  <child link="arm_base_v2_1"/>
+</joint>
 <joint name="joint1" type="revolute">
   <origin xyz="-0.005751 0.088 0.13" rpy="0 0 0"/>
@@ -123,8 +128,3 @@
   <axis xyz="-1.0 -0.0 0.0"/>
 </joint>
-<joint name="fix" type="fixed">
-  <origin xyz="0.0 0.0 0.0" rpy="0 0 0"/>
-  <parent link="base_link"/>
-  <child link="arm_base_v2_1"/>
-</joint>
 </robot>

Commit message: ide_arm_descriptionとnhk2026_simのためのURDFモデルとlaunchファイルを追加し、メッシュファイルを更新

File: src/ide_arm_description/urdf/ide_arm.xacro (robot description, xacro)
@@ -12,5 +12,5 @@
     <origin xyz="0 0 0" rpy="0 0 0"/>
     <geometry>
-      <mesh filename="package://ide_arm_description/meshes/base_link.stl" scale="1.0 1.0 1.0"/>
+      <mesh filename="package://ide_arm_description/meshes/base_link_ide_arm.stl" scale="1.0 1.0 1.0"/>
     </geometry>
     <material name="_"/>
@@ -19,5 +19,5 @@
     <origin xyz="0 0 0" rpy="0 0 0"/>
     <geometry>
-      <mesh filename="package://ide_arm_description/meshes/base_link.stl" scale="1.0 1.0 1.0"/>
+      <mesh filename="package://ide_arm_description/meshes/base_link_ide_arm.stl" scale="1.0 1.0 1.0"/>
     </geometry>
   </collision>
