Commit message: base_linkをbase_link_r2に変更し、関連するメッシュファイルを追加

File: src/r2_step_climber_description/urdf/r2_step_climber.xacro (robot description, xacro)
@@ -3,5 +3,5 @@
 <xacro:include filename="$(find r2_step_climber_description)/urdf/materials.xacro" />
 <xacro:include filename="$(find r2_step_climber_description)/urdf/r2_step_climber.trans" />
-<link name="base_link">
+<link name="base_link_r2">
   <inertial>
     <origin xyz="-0.01026966368511183 -0.08711294351843835 0.11765235493872747" rpy="0 0 0"/>
@@ -12,5 +12,5 @@
     <origin xyz="0 0 0" rpy="0 0 0"/>
     <geometry>
-      <mesh filename="package://r2_step_climber_description/meshes/base_link.stl" scale="0.001 0.001 0.001"/>
+      <mesh filename="package://r2_step_climber_description/meshes/base_link_r2.stl" scale="0.001 0.001 0.001"/>
     </geometry>
     <material name="_"/>
@@ -19,5 +19,5 @@
     <origin xyz="0 0 0" rpy="0 0 0"/>
     <geometry>
-      <mesh filename="package://r2_step_climber_description/meshes/base_link.stl" scale="0.001 0.001 0.001"/>
+      <mesh filename="package://r2_step_climber_description/meshes/base_link_r2.stl" scale="0.001 0.001 0.001"/>
     </geometry>
   </collision>
@@ -85,5 +85,5 @@
 <joint name="back_arm_joint" type="revolute">
   <origin xyz="0.019 -0.31 0.06" rpy="0 0 0"/>
-  <parent link="base_link"/>
+  <parent link="base_link_r2"/>
   <child link="R2_step_clibmer_arm_v2_1"/>
   <axis xyz="-1.0 0.0 0.0"/>
@@ -92,5 +92,5 @@
 <joint name="left_arm_joint" type="continuous">
   <origin xyz="-0.275 0.095 0.06" rpy="0 0 0"/>
-  <parent link="base_link"/>
+  <parent link="base_link_r2"/>
   <child link="R2_step_climber_front_v2_1"/>
   <axis xyz="-1.0 0.0 0.0"/>
@@ -98,5 +98,5 @@
 <joint name="right_arm_joint" type="continuous">
   <origin xyz="0.275 0.095 0.06" rpy="0 0 0"/>
-  <parent link="base_link"/>
+  <parent link="base_link_r2"/>
   <child link="R2_step_climber_front_v2_2"/>
   <axis xyz="1.0 0.0 0.0"/>

Commit message: base_root_r2リンクとジョイントを追加し、left_arm_jointの回転を修正

File: src/r2_step_climber_description/urdf/r2_step_climber.xacro (robot description, xacro)
@@ -3,4 +3,5 @@
 <xacro:include filename="$(find r2_step_climber_description)/urdf/materials.xacro" />
 <xacro:include filename="$(find r2_step_climber_description)/urdf/r2_step_climber.trans" />
+<link name="base_root_r2"/>
 <link name="base_link_r2">
   <inertial>
@@ -83,4 +84,8 @@
   </collision>
 </link>
+<joint name="base_root_r2" type="fixed">
+  <parent link="base_root_r2"/>
+  <child link="base_link_r2"/>
+</joint>
 <joint name="back_arm_joint" type="revolute">
   <origin xyz="0.019 -0.31 0.06" rpy="0 0 0"/>
@@ -91,5 +96,5 @@
 </joint>
 <joint name="left_arm_joint" type="continuous">
-  <origin xyz="-0.275 0.095 0.06" rpy="0 0 0"/>
+  <origin xyz="-0.275 0.095 0.06" rpy="3.141593 0 0"/>
   <parent link="base_link_r2"/>
   <child link="R2_step_climber_front_v2_1"/>
@@ -100,5 +105,5 @@
   <parent link="base_link_r2"/>
   <child link="R2_step_climber_front_v2_2"/>
-  <axis xyz="1.0 0.0 0.0"/>
+  <axis xyz="-1.0 0.0 0.0"/>
 </joint>
 </robot>
